Commit message: lidar gazebo

File: description/robot.urdf.xacro (robot description, xacro)
@@ -3,3 +3,4 @@
     <xacro:include filename="robot_core.xacro" />
     <xacro:include filename="gazebo_control.xacro"/>
+    <xacro:include filename="lidar.xacro"/>
 </robot>

File: description/robot_core.xacro (robot description, xacro)
@@ -31,4 +31,7 @@
         <color rgba="1 0 0 1"/>
     </material>
+    <material name="yellow">
+        <color rgba="1 1 0 1"/>
+    </material>
     <!-- BASE LINK -->
     <link name="base_link">
@@ -54,5 +57,5 @@
                 <box size="${chassis_length} ${chassis_width} ${chassis_height}"/>
             </geometry>
-            <material name="orange"/>
+            <material name="white"/>
         </visual>
         <collision>
